File: romext-2364/kicad/romext-2364.kicad_sch (KiCad schematic)
At the start: 0 parts

Commit message: romext-2364 sch: Add 2764 from standard KiCad library
Parts:
- added U1: 2764, Package_DIP:DIP-28_W15.24mm, symbol Memory_EPROM:2764
Changed lines of the file:
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@@
 	(generator_version "9.0")
 	(paper "A4")
+	(symbol
+		(lib_id "Memory_EPROM:2764")
+		(at 143.51 83.82 0)
+		(unit 1)
+		(exclude_from_sim no)
+		(in_bom yes)
+		(on_board yes)
+		(dnp no)
+		(fields_autoplaced yes)
+		(property "Reference" "U1"
+			(at 145.6533 55.88 0)
+			(effects
+				(font
+					(size 1.27 1.27)
+				)
+				(justify left)
+			)
+		)
+		(property "Value" "2764"
+			(at 145.6533 58.42 0)
+			(effects
+				(font
+					(size 1.27 1.27)
+				)
+				(justify left)
+			)
+		)
+		(property "Footprint" "Package_DIP:DIP-28_W15.24mm"
+			(at 143.51 83.82 0)
+			(effects
+				(font
+					(size 1.27 1.27)
+				)
+				(hide yes)
+			)
+		)
+		(property "Datasheet" "https://downloads.reactivemicro.com/Electronics/ROM/2764%20EPROM.pdf"
+			(at 143.51 83.82 0)
+			(effects
+				(font
+					(size 1.27 1.27)
+				)
+				(hide yes)
+			)
+		)
+		(property "Description" "EPROM 64 KiBit, [Obsolete 2000-11]"
+			(at 143.51 83.82 0)
+			(effects
+				(font
+					(size 1.27 1.27)
+				)
+				(hide yes)
+			)
+		)
+		(pin "12"
+		)
+		(pin "17"
+		)
+		(pin "3"
+		)
+		(pin "9"
+		)
+		(pin "14"
+		)
+		(pin "10"
+		)
+		(pin "15"
+		)
+		(pin "18"
+		)
+		(pin "5"
+		)
+		(pin "28"
+		)
+		(pin "6"
+		)
+		(pin "8"
+		)
+		(pin "11"
+		)
+		(pin "7"
+		)
+		(pin "20"
+		)
+		(pin "22"
+		)
+		(pin "4"
+		)
+		(pin "26"
+		)
+		(pin "16"
+		)
+		(pin "13"
+		)
+		(pin "25"
+		)
+		(pin "1"
+		)
+		(pin "19"
+		)
+		(pin "2"
+		)
+		(pin "24"
+		)
+		(pin "23"
+		)
+		(pin "21"
+		)
+		(pin "27"
+		)
+		(instances
+			(project ""
+				(path "/a4f6bc9b-0965-4439-8426-46811e7c40b1"
+					(reference "U1")
+					(unit 1)
+				)
+			)
+		)
+	)
 	(sheet_instances
 		(path "/"
