File: romext-2364/kicad/romext-2364.kicad_sch (KiCad schematic)
At the start: 0 parts

Commit message: romext-2364 sch: Complete schematic of basic version
The "2364" is actually a socket J1, where the addr/data/select
lines are outputs because this is wired to the socket on the
PC-8001 motherboard.

This is the simplest design that will work with the PC-8001 and
an ST Microelectronics M2764A; it does not yet provide facilities
to work with systems or EPROMs that vary how they use chip select
or have different requirements for levels on the programming pins
during read operations.
Parts:
- added J1: 2364, Package_DIP:DIP-24_W15.24mm, symbol 0cjs-hwdev:2364
- added U1: 2764, Package_DIP:DIP-28_W15.24mm, symbol Memory_EPROM:2764
Connections:
- new net: J1.20 (~{CS}), U1.20 (~{CE}), U1.22 (~{OE})
- new net A0: J1.8 (A0), U1.10 (A0)
- new net A1: J1.7 (A1), U1.9 (A1)
- new net A10: J1.19 (A10), U1.21 (A10)
- new net A11: J1.18 (A11), U1.23 (A11)
- new net A12: J1.21 (A12), U1.2 (A12)
- new net A2: J1.6 (A2), U1.8 (A2)
- new net A3: J1.5 (A3), U1.7 (A3)
- new net A4: J1.4 (A4), U1.6 (A4)
- new net A5: J1.3 (A5), U1.5 (A5)
- new net A6: J1.2 (A6), U1.4 (A6)
- new net A7: J1.1 (A7), U1.3 (A7)
- new net A8: J1.23 (A8), U1.25 (A8)
- new net A9: J1.22 (A9), U1.24 (A9)
- new net D0: J1.9 (D0), U1.11 (D0)
- new net D1: J1.10 (D1), U1.12 (D1)
- new net D2: J1.11 (D2), U1.13 (D2)
- new net D3: J1.13 (D3), U1.15 (D3)
- new net D4: J1.14 (D4), U1.16 (D4)
- new net D5: J1.15 (D5), U1.17 (D5)
- new net D6: J1.16 (D6), U1.18 (D6)
- new net D7: J1.17 (D7), U1.19 (D7)
- new net GND: J1.12 (GND), U1.14 (GND)
- new net VCC: J1.24 (Vcc), U1.1 (VPP), U1.27 (~{PGM}), U1.28 (VCC)

Commit message: hwdev.romext-2364: Add name, url and revision to title block
Other:
- title: (none) -> romext-2364
Changed lines of the file:
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@@
 	(generator_version "9.0")
 	(paper "A4")
+	(title_block
+		(title "romext-2364")
+		(rev "1")
+		(comment 1 "https://github.com/0cjs/hwdev")
+	)
 	(junction
 		(at 154.94 105.41)

Commit message: romext-2364 pcb: Change U1/2764 to use standard library ZIF footprint
Bumps PCB revision to 1-2dev.

The footprint was hard to find[1]; one has to turn off the footprint
filter to have it come up.

This updates the schematic as well, but just the footprint assignment
in it, so we don't need to bump the revision. (It does update the PDF,
however, because that contains the footprint info in the internal
Javascript for popups or whatever.)

[1]: https://forum.kicad.info/t/please-add-zif-to-the-descriptions-of-zero-insertion-force-sockets/62549/6
Parts:
- U1: footprint Package_DIP:DIP-28_W15.24mm -> Socket:DIP_Socket-28_W11.9_W12.7_W15.24_W17.78_W18.5_3M_228-1277-00-0602J
Changed lines of the file:
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@@
 			)
 		)
-		(property "Footprint" "Package_DIP:DIP-28_W15.24mm"
+		(property "Footprint" "Socket:DIP_Socket-28_W11.9_W12.7_W15.24_W17.78_W18.5_3M_228-1277-00-0602J"
 			(at 165.1 90.17 0)
 			(effects
