File: rom-read-adapter/kicad/rom-read-adapter.kicad_sch (KiCad schematic)
At the start: 27 parts

Commit message: rom-read-adapter sch: Assign all footprints but ZIF
We can't assign the ZIF yet as we have no footprint for it.
Parts:
- C1: footprint (none) -> Capacitor_THT:C_Disc_D5.1mm_W3.2mm_P5.00mm
- JH1: footprint (none) -> Connector_PinHeader_2.54mm:PinHeader_2x25_P2.54mm_Vertical
- JH11, JH12, JH13, JH14, JH15, JH21, JH22, JH23, JH24, JH31, JH32, JH33, JH34, JH41, JH42, JH43, JH44: footprint (none) -> Connector_PinHeader_2.54mm:PinHeader_1x04_P2.54mm_Vertical
- JH2: footprint (none) -> Connector_PinHeader_2.54mm:PinHeader_1x13_P2.54mm_Vertical
- JH3: footprint (none) -> Connector_PinHeader_2.54mm:PinHeader_1x05_P2.54mm_Vertical
- JH4: footprint (none) -> Connector_PinHeader_2.54mm:PinHeader_1x02_P2.54mm_Vertical
- JH5: footprint (none) -> Connector_PinHeader_2.54mm:PinHeader_1x03_P2.54mm_Vertical
- JH6: footprint (none) -> Connector_PinHeader_2.54mm:PinHeader_1x01_P2.54mm_Vertical
- JR2, JR3: footprint (none) -> Connector_PinHeader_2.54mm:PinHeader_1x24_P2.54mm_Vertical
Changed lines of the file:
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@@
 			)
 		)
-		(property "Footprint" ""
+		(property "Footprint" "Connector_PinHeader_2.54mm:PinHeader_1x04_P2.54mm_Vertical"
 			(at 157.48 134.62 0)
 			(effects
@@
 			)
 		)
-		(property "Footprint" ""
+		(property "Footprint" "Connector_PinHeader_2.54mm:PinHeader_1x04_P2.54mm_Vertical"
 			(at 132.08 134.62 0)
 			(effects
@@
 			)
 		)
-		(property "Footprint" ""
+		(property "Footprint" "Connector_PinHeader_2.54mm:PinHeader_1x24_P2.54mm_Vertical"
 			(at 153.67 95.25 0)
 			(effects
@@
 			)
 		)
-		(property "Footprint" ""
+		(property "Footprint" "Connector_PinHeader_2.54mm:PinHeader_1x04_P2.54mm_Vertical"
 			(at 101.6 90.17 0)
 			(effects
@@
 			)
 		)
-		(property "Footprint" ""
+		(property "Footprint" "Connector_PinHeader_2.54mm:PinHeader_1x04_P2.54mm_Vertical"
 			(at 175.26 105.41 0)
 			(effects
@@
 			)
 		)
-		(property "Footprint" ""
+		(property "Footprint" "Connector_PinHeader_2.54mm:PinHeader_1x04_P2.54mm_Vertical"
 			(at 162.56 53.34 0)
 			(effects
@@
 			)
 		)
-		(property "Footprint" ""
+		(property "Footprint" "Connector_PinHeader_2.54mm:PinHeader_1x04_P2.54mm_Vertical"
 			(at 149.86 53.34 0)
 			(effects
@@
 			)
 		)
-		(property "Footprint" ""
+		(property "Footprint" "Connector_PinHeader_2.54mm:PinHeader_1x04_P2.54mm_Vertical"
 			(at 101.6 120.65 0)
 			(effects
@@
 			)
 		)
-		(property "Footprint" ""
+		(property "Footprint" "Connector_PinHeader_2.54mm:PinHeader_1x04_P2.54mm_Vertical"
 			(at 101.6 105.41 0)
 			(effects
@@
 			)
 		)
-		(property "Footprint" ""
+		(property "Footprint" "Connector_PinHeader_2.54mm:PinHeader_1x04_P2.54mm_Vertical"
 			(at 175.26 74.93 0)
 			(effects
@@
 			)
 		)
-		(property "Footprint" ""
+		(property "Footprint" "Connector_PinHeader_2.54mm:PinHeader_1x04_P2.54mm_Vertical"
 			(at 101.6 74.93 0)
 			(effects
@@
 			)
 		)
-		(property "Footprint" ""
+		(property "Footprint" "Connector_PinHeader_2.54mm:PinHeader_1x13_P2.54mm_Vertical"
 			(at 120.65 107.95 0)
 			(effects
@@
 			)
 		)
-		(property "Footprint" ""
+		(property "Footprint" "Connector_PinHeader_2.54mm:PinHeader_1x04_P2.54mm_Vertical"
 			(at 175.26 90.17 0)
 			(effects
@@
 			)
 		)
-		(property "Footprint" ""
+		(property "Footprint" "Connector_PinHeader_2.54mm:PinHeader_1x04_P2.54mm_Vertical"
 			(at 144.78 134.62 0)
 			(effects
@@
 			)
 		)
-		(property "Footprint" ""
+		(property "Footprint" "Connector_PinHeader_2.54mm:PinHeader_1x03_P2.54mm_Vertical"
 			(at 156.21 97.79 0)
 			(effects
@@
 			)
 		)
-		(property "Footprint" ""
+		(property "Footprint" "Connector_PinHeader_2.54mm:PinHeader_1x02_P2.54mm_Vertical"
 			(at 156.21 107.95 0)
 			(effects
@@
 			)
 		)
-		(property "Footprint" ""
+		(property "Footprint" "Connector_PinHeader_2.54mm:PinHeader_1x04_P2.54mm_Vertical"
 			(at 111.76 53.34 0)
 			(effects
@@
 			)
 		)
-		(property "Footprint" ""
+		(property "Footprint" "Connector_PinHeader_2.54mm:PinHeader_1x04_P2.54mm_Vertical"
 			(at 137.16 53.34 0)
 			(effects
@@
 			)
 		)
-		(property "Footprint" ""
+		(property "Footprint" "Capacitor_THT:C_Disc_D5.1mm_W3.2mm_P5.00mm"
 			(at 160.9852 73.66 0)
 			(effects
@@
 			)
 		)
-		(property "Footprint" ""
+		(property "Footprint" "Connector_PinHeader_2.54mm:PinHeader_1x04_P2.54mm_Vertical"
 			(at 175.26 120.65 0)
 			(effects
@@
 			)
 		)
-		(property "Footprint" ""
+		(property "Footprint" "Connector_PinHeader_2.54mm:PinHeader_1x04_P2.54mm_Vertical"
 			(at 124.46 53.34 0)
 			(effects
@@
 			)
 		)
-		(property "Footprint" ""
+		(property "Footprint" "Connector_PinHeader_2.54mm:PinHeader_1x24_P2.54mm_Vertical"
 			(at 123.19 92.71 0)
 			(effects
@@
 			)
 		)
-		(property "Footprint" ""
+		(property "Footprint" "Connector_PinHeader_2.54mm:PinHeader_1x01_P2.54mm_Vertical"
 			(at 156.21 90.17 0)
 			(effects
@@
 			)
 		)
-		(property "Footprint" ""
+		(property "Footprint" "Connector_PinHeader_2.54mm:PinHeader_2x25_P2.54mm_Vertical"
 			(at 60.96 93.98 0)
 			(effects
@@
 			)
 		)
-		(property "Footprint" ""
+		(property "Footprint" "Connector_PinHeader_2.54mm:PinHeader_1x04_P2.54mm_Vertical"
 			(at 119.38 134.62 0)
 			(effects
@@
 			)
 		)
-		(property "Footprint" ""
+		(property "Footprint" "Connector_PinHeader_2.54mm:PinHeader_1x05_P2.54mm_Vertical"
 			(at 156.21 118.11 0)
 			(effects

Commit message: rom-read-adapter sch: ZIF symbol update from lib and footprint; pin updates
The pin updates are for JR3 (the pin header connected directly to ZIF
pins 25-48) where we had pins numbered from 25-48 on JR3 also numbered
to match. Not clear if this was a problem, because we also had the
connections between the ZIF and this header in a real mess, but it's
now exactly pin-to-pin as it should always have been. Before we
weren't seeing the correct connections on the PCB editor ratsnest; now
we are.
Parts:
- JR1: footprint (none) -> 0cjs_hwdev:DIP_Socket-48_W11.9_W12.7_W15.24_W17.78_W18.5
Connections:
- net at JR1.25 (Pin_25): now also JR3.1 (Pin_25); no longer JR3.25 (Pin_1)
- net at JR1.26 (Pin_26): now also JR3.2 (Pin_26); no longer JR3.26 (Pin_2)
- net at JR1.27 (Pin_27): now also JR3.3 (Pin_27); no longer JR3.27 (Pin_3)
- net at JR1.29 (Pin_29): now also JR3.5 (Pin_29); no longer JR3.29 (Pin_5)
- net at JR1.30 (Pin_30): now also JR3.6 (Pin_30); no longer JR3.30 (Pin_6)
- net at JR1.31 (Pin_31): now also JR3.7 (Pin_31); no longer JR3.31 (Pin_7)
- net at JR1.32 (Pin_32): now also JR3.8 (Pin_32); no longer JR3.32 (Pin_8)
- net at JR1.33 (Pin_33): now also JR3.9 (Pin_33); no longer JR3.33 (Pin_9)
- net at JR1.34 (Pin_34): now also JR3.10 (Pin_34); no longer JR3.34 (Pin_10)
- net at JR1.35 (Pin_35): now also JR3.11 (Pin_35); no longer JR3.35 (Pin_11)
- net at JR1.36 (Pin_36): now also JR3.12 (Pin_36); no longer JR3.36 (Pin_12)
- net at JR1.37 (Pin_37): now also JR3.13 (Pin_37); no longer JR3.37 (Pin_13)
- net at JR1.38 (Pin_38): now also JR3.14 (Pin_38); no longer JR3.38 (Pin_14)
- net at JR1.39 (Pin_39): now also JR3.15 (Pin_39); no longer JR3.39 (Pin_15)
- net at JR1.40 (Pin_40): now also JR3.16 (Pin_40); no longer JR3.40 (Pin_16)
- net at JR1.41 (Pin_41): now also JR3.17 (Pin_41); no longer JR3.41 (Pin_17)
- net at JR1.42 (Pin_42): now also JR3.18 (Pin_42); no longer JR3.42 (Pin_18)
- net at JR1.43 (Pin_43): now also JR3.19 (Pin_43); no longer JR3.43 (Pin_19)
- net at JR1.44 (Pin_44): now also JR3.20 (Pin_44); no longer JR3.44 (Pin_20)
- net at JR1.45 (Pin_45): now also JR3.21 (Pin_45); no longer JR3.45 (Pin_21)
- net at JR1.46 (Pin_46): now also JR3.22 (Pin_46); no longer JR3.46 (Pin_22)
- net at JR1.47 (Pin_47): now also JR3.23 (Pin_47); no longer JR3.47 (Pin_23)
- net at JR1.48 (Pin_48): now also JR3.24 (Pin_48); no longer JR3.48 (Pin_24)
- new net: JR1.28 (Pin_28), JR3.4 (Pin_28)
Changed lines of the file:
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@@
 			)
 		)
-		(property "Footprint" ""
+		(property "Footprint" "0cjs_hwdev:DIP_Socket-48_W11.9_W12.7_W15.24_W17.78_W18.5"
 			(at 138.43 93.98 0)
 			(effects
@@
 		)
 		(pin "1"
-		)
-		(pin ""
 		)
 		(pin "30"
@@
 			)
 		)
-		(pin "33"
-		)
-		(pin "34"
-		)
-		(pin "31"
-		)
-		(pin "44"
-		)
-		(pin "41"
-		)
-		(pin "27"
-		)
-		(pin "35"
-		)
-		(pin "30"
-		)
-		(pin "43"
-		)
-		(pin "29"
-		)
-		(pin "26"
-		)
-		(pin "38"
-		)
-		(pin "45"
-		)
-		(pin "40"
-		)
-		(pin "39"
-		)
-		(pin "47"
-		)
-		(pin "25"
-		)
-		(pin "48"
-		)
-		(pin "36"
-		)
-		(pin "37"
-		)
-		(pin "42"
-		)
-		(pin "46"
-		)
-		(pin "28"
-		)
-		(pin "32"
-		)
-		(instances
+		(pin "19"
+		)
+		(pin "8"
+		)
+		(pin "15"
+		)
+		(pin "20"
+		)
+		(pin "21"
+		)
+		(pin "2"
+		)
+		(pin "18"
+		)
+		(pin "4"
+		)
+		(pin "16"
+		)
+		(pin "22"
+		)
+		(pin "1"
+		)
+		(pin "5"
+		)
+		(pin "13"
+		)
+		(pin "24"
+		)
+		(pin "17"
+		)
+		(pin "11"
+		)
+		(pin "3"
+		)
+		(pin "10"
+		)
+		(pin "7"
+		)
+		(pin "12"
+		)
+		(pin "9"
+		)
+		(pin "23"
+		)
+		(pin "14"
+		)
+		(pin "6"
+		)
+		(instances

Commit message: WIP rom-read-adapter: Replace disc cap with axial; all traces routed
We've gone with the solution mentioned in the previous commit message,
where we put an axial cap kinda-near the GND and VCC pins in the work
area. It could be closer, by moving some traces, or even by putting it
in between the socket pin connectors, though that would cover up lots
of pin numbers. (Maybe try it on the bottom? Still would moving some
traces to make room for the pads.)
Parts:
- C1: footprint Capacitor_THT:C_Disc_D5.1mm_W3.2mm_P5.00mm -> Capacitor_THT:C_Axial_L3.8mm_D2.6mm_P10.00mm_Horizontal
Changed lines of the file:
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@@
 			)
 		)
-		(property "Footprint" "Capacitor_THT:C_Disc_D5.1mm_W3.2mm_P5.00mm"
+		(property "Footprint" "Capacitor_THT:C_Axial_L3.8mm_D2.6mm_P10.00mm_Horizontal"
 			(at 160.9852 73.66 0)
 			(effects
