File: rom-read-adapter/kicad/rom-read-adapter.kicad_pcb (KiCad board)
At the start: 2 copper layers, 100 x 100 mm, 31 parts

Commit message: rom-read-adapter: Fully routed again. Lots of warnings to clean up.
Removed warnings:
- Courtyard overlaps for jumperable header pins in work area.
Parts:
- moved C1 11.5 mm to (190.5, 113.1)
Routing:
- net GND: track 438.1 -> 168.9 mm, vias 2 -> 1
- net D7: track 369.5 -> 167.0 mm
- net Net-(JR1-Pin_41): track 234.7 -> 59.5 mm
- net Net-(JR1-Pin_16): track 218.1 -> 56.6 mm, vias 3 -> 1
- net Net-(JR1-Pin_43): track 201.7 -> 57.4 mm
- net Net-(JR1-Pin_14): track 179.5 -> 54.5 mm
- net D6: track 68.6 -> 160.2 mm
- net Net-(JR1-Pin_9): track 143.2 -> 56.0 mm
- net A10: track 17.6 -> 92.7 mm, vias 0 -> 1
- net A9: track 15.0 -> 84.2 mm, vias 0 -> 1
- net A8: track 18.6 -> 86.9 mm, vias 0 -> 1
- net Net-(JR1-Pin_39): track 1.79 -> 61.6 mm
- net Net-(JR1-Pin_38): track 1.79 -> 59.5 mm
- net A12: track 18.6 -> 73.3 mm, vias 0 -> 1
- net Net-(JR1-Pin_42): track 4.76 -> 58.5 mm
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